Commit message: teleop: adopt the official Maker URDF and drive its gripper
- Replace the hand-built URDF with the SDK's
- From makermods-robotics/maker-arm-sdk at commit b30d05a
- 52 STL meshes, all referenced
- Add revision_report.json for provenance
- Real gripper joint: left drives, right mimics
- Map the gripper motor angle to metres
- Gripper curve is visual-preview only
- Keep the model Y-up (up "+Y")
- Ignore the URDF's unverified joint limits
- Pass ignore-limits through createUrdfViewer
- Add a trailing newline per the hook
- Update the Maker URDF mapping tests

File: frontend/public/maker-urdf/robot.urdf (robot description, URDF)
Before this commit: robot generated_robot, 7 links, 6 joints
Links:
- added link grasp_center
- added link gripper_left, mass 0.0599060506559; collision mesh filename=meshes/part_031_solid_031.stl scale=0.001 0.001 0.001; collision mesh filename=meshes/part_032_solid_032.stl scale=0.001 0.001 0.001
- added link gripper_right, mass 0.0596144977418; collision mesh filename=meshes/part_038_solid_038.stl scale=0.001 0.001 0.001; collision mesh filename=meshes/part_039_solid_039.stl scale=0.001 0.001 0.001
- link link_007: mass 0.4 -> 0.280479451602; geometry collision mesh filename=meshes/part_022_solid_022.stl scale=0.001 0.001 0.001; collision mesh filename=meshes/part_026_solid_026.stl scale=0.001 0.001 0.001
Joints:
- added joint grasp_center_joint: type fixed, parent link_007, child grasp_center, origin xyz=-3.17806289618e-09 -1.25735103017e-08 -0.169638704618 rpy=0 0 0
- added joint gripper_left_joint: type prismatic, parent link_007, child gripper_left, origin xyz=0 0 0 rpy=0 0 0, axis 7.2798028557e-08 1 4.65288500486e-09, limit lower=0 upper=0.0524125 effort=20 velocity=0.1
- added joint gripper_right_joint: type prismatic, parent link_007, child gripper_right, origin xyz=0 0 0 rpy=0 0 0, axis -7.2798028557e-08 -1 -4.65288500486e-09, limit lower=0 upper=0.0524125 effort=20 velocity=0.1, mimic joint=gripper_left_joint multiplier=1 offset=0
- joint link_002_joint: limit lower=-2.76111 upper=2.72446 effort=10 velocity=5 -> lower=-2.8 upper=2.8 effort=10 velocity=5
- joint link_003_joint: limit lower=-3.05956 upper=-0.05585 effort=10 velocity=5 -> lower=-3.14 upper=0 effort=10 velocity=5
- joint link_004_joint: limit lower=0.04887 upper=4.12072 effort=10 velocity=5 -> lower=0 upper=3.14 effort=10 velocity=5
- joint link_005_joint: limit lower=-1.13795 upper=1.81514 effort=10 velocity=5 -> lower=-1.6 upper=1.73 effort=10 velocity=5
- joint link_006_joint: limit lower=-1.70344 upper=1.36136 effort=10 velocity=5 -> lower=-1.57 upper=1.57 effort=10 velocity=5
- joint link_007_joint: limit lower=-2.67384 upper=2.6529 effort=10 velocity=5 -> lower=-2.7 upper=2.7 effort=10 velocity=5

Commit message: Use fitted Maker Arm inertials and joint friction

File: frontend/public/maker-urdf/robot.urdf (robot description, URDF)
Before this commit: robot maker_arm_gripper_v1, 10 links, 9 joints
Links:
- link gripper_left: mass 0.0599060506559 -> 0.069790549
- link gripper_right: mass 0.0596144977418 -> 0.06945089
- link link_004: mass 0.6 -> 0.9018
- link link_005: mass 0.4 -> 0.466
- link link_006: mass 0.35 -> 0.40775
- link link_007: mass 0.280479451602 -> 0.32675856
